Commit message: default_pick_and_place.py

File: ur5_with_robotiq_gripper/icl_ur5_setup_description/robots/ur5_robotiq_85_joint_limited.xacro (robot description, xacro)
@@ -58,5 +58,5 @@
       <parent link="${prefix}wrist_3_link"/>
       <child link="realsense_link"/>
-      <origin xyz="0 0.06 0.01" rpy="0 -1.5708 1.5708"/>
+      <origin xyz="0 0.06 0.01" rpy="0.0 -1.5708 1.5708"/>
     </joint>
     <!-- <link name="${prefix}tool" />

Commit message: apriltag detection + Pick and place using UR5 with Robotiq 2F-85 gripper

File: ur5_with_robotiq_gripper/icl_ur5_setup_description/robots/ur5_robotiq_85_joint_limited.xacro (robot description, xacro)
@@ -33,4 +33,13 @@
       <origin xyz=" 0.0 0.0 0.0" rpy="0.0 0.0 ${pi/2}" />
     </joint>
+    <!-- TCP (Tool Center Point) - gripper finger tips grasp point -->
+    <!-- This represents where objects should be positioned for grasping -->
+    <link name="${prefix}gripper_tcp"/>
+    <joint name="gripper_tcp_joint" type="fixed">
+      <parent link="${prefix}tool0"/>
+      <child link="${prefix}gripper_tcp"/>
+      <!-- Robotiq 85: ~17cm from tool0 to finger tips when fingers are centered -->
+      <origin xyz="0 0 0.17" rpy="0 0 0"/>
+    </joint>
     <!-- Camera link -->
     <link name="realsense_link">
@@ -59,4 +68,15 @@
       <child link="realsense_link"/>
       <origin xyz="0 0.06 0.01" rpy="0.0 -1.5708 1.5708"/>
+    </joint>
+    <!-- Optical frame for camera (ROS optical convention: X=right, Y=down, Z=forward) -->
+    <link name="realsense_color_optical_frame"/>
+    <joint name="realsense_optical_joint" type="fixed">
+      <parent link="realsense_link"/>
+      <child link="realsense_color_optical_frame"/>
+      <!-- Rotate from camera body frame to optical frame:
+           Camera body: X=forward, Y=left, Z=up
+           Optical: X=right, Y=down, Z=forward
+           Rotation: -pi/2 around X, then -pi/2 around Z -->
+      <origin xyz="0 0 0" rpy="-1.5708 0 -1.5708"/>
     </joint>
     <!-- <link name="${prefix}tool" />
@@ -91,5 +111,6 @@
         <imageTopicName>camera/image_raw</imageTopicName>
         <cameraInfoTopicName>camera/camera_info</cameraInfoTopicName>
-        <frameName>realsense_link</frameName>
+        <frameName>realsense_color_optical_frame</frameName>
+        <hackBaseline>0.07</hackBaseline>
       </plugin>
     </sensor>

Commit message: feat: Enhance UR5 + Robotiq integration with AprilTag detection and Gazebo improvements
- Added runtime dependencies to `icl_ur5_setup_bringup/package.xml` for ROS nodes.
- Updated `icl_ur5_setup_description/package.xml` to include `gazebo_ros` for proper path resolution.
- Integrated a Realsense camera into the UR5 model using a macro in `realsense.xacro`, consolidating camera definitions.
- Implemented a grasp-fix plugin in the URDF to improve gripper reliability in Gazebo.
- Modified the Gazebo world file to include a dynamic cube and a stable shelf for better interaction.
- Created a Docker setup for development on Ubuntu 22.04, including a comprehensive `Dockerfile` and `docker-compose.yml`.
- Added scripts for building the workspace and managing the Docker container environment.
- Updated the gripper controller configuration to use position control for better performance.
- Introduced a `.gitignore` file to exclude build artifacts and editor-specific files.

File: ur5_with_robotiq_gripper/icl_ur5_setup_description/robots/ur5_robotiq_85_joint_limited.xacro (robot description, xacro)
@@ -5,4 +5,5 @@
   <xacro:include filename="$(find ur_description)/urdf/ur5.xacro" />
   <xacro:include filename="$(find icl_ur5_setup_description)/urdf/robotiq_arg2f_85_model_macro.xacro" />
+  <xacro:include filename="$(find icl_ur5_setup_description)/urdf/realsense.xacro" />
   <!-- <xacro:include filename="$(find icl_ur5_setup_description)/urdf/robotiq_fts300.urdf.xacro" /> -->
   <xacro:macro name="ur5_with_gripper_joint_limited" params="prefix">
@@ -42,42 +43,6 @@
       <origin xyz="0 0 0.17" rpy="0 0 0"/>
     </joint>
-    <!-- Camera link -->
-    <link name="realsense_link">
-      <visual>
-        <geometry>
-          <box size="0.04 0.04 0.025"/>
-        </geometry>
-        <material name="gray">
-          <color rgba="0.5 0.5 0.5 1"/>
-        </material>
-      </visual>
-      <collision>
-        <geometry>
-          <box size="0.04 0.04 0.025"/>
-        </geometry>
-      </collision>
-      <inertial>
-        <mass value="0.07"/>
-        <origin xyz="0 0 0" rpy="0 0 0"/>
-        <inertia ixx="0.0001" ixy="0.0" ixz="0.0" iyy="0.0001" iyz="0.0" izz="0.0001"/>
-      </inertial>
-    </link>
-    <!-- Fixed joint to attach camera to wrist_3_link, offset up and forward -->
-    <joint name="realsense_joint" type="fixed">
-      <parent link="${prefix}wrist_3_link"/>
-      <child link="realsense_link"/>
-      <origin xyz="0 0.06 0.01" rpy="0.0 -1.5708 1.5708"/>
-    </joint>
-    <!-- Optical frame for camera (ROS optical convention: X=right, Y=down, Z=forward) -->
-    <link name="realsense_color_optical_frame"/>
-    <joint name="realsense_optical_joint" type="fixed">
-      <parent link="realsense_link"/>
-      <child link="realsense_color_optical_frame"/>
-      <!-- Rotate from camera body frame to optical frame:
-           Camera body: X=forward, Y=left, Z=up
-           Optical: X=right, Y=down, Z=forward
-           Rotation: -pi/2 around X, then -pi/2 around Z -->
-      <origin xyz="0 0 0" rpy="-1.5708 0 -1.5708"/>
-    </joint>
+    <!-- Wrist-mounted depth (RGB-D) camera — defined in realsense.xacro -->
+    <xacro:realsense_camera parent="${prefix}wrist_3_link"/>
     <!-- <link name="${prefix}tool" />
     <joint name="tool_tip" type="fixed">
@@ -88,31 +53,31 @@
   </xacro:macro>
   <xacro:ur5_with_gripper_joint_limited prefix=""/>
- <!-- Camera Plugin -->
-  <gazebo reference="realsense_link">
-    <sensor type="camera" name="realsense_camera">
-      <always_on>true</always_on>
-      <update_rate>30</update_rate>
-      <visualize>true</visualize>
-      <camera>
-        <horizontal_fov>1.3962634</horizontal_fov>
-        <image>
-          <width>640</width>
-          <height>480</height>
-          <format>R8G8B8</format>
-        </image>
-        <clip>
-          <near>0.1</near>
-          <far>5.0</far>
-        </clip>
-      </camera>
-      <plugin name="realsense_camera_controller" filename="libgazebo_ros_camera.so">
-        <robotNamespace>/ur5</robotNamespace>
-        <cameraName>realsense</cameraName>
-        <imageTopicName>camera/image_raw</imageTopicName>
-        <cameraInfoTopicName>camera/camera_info</cameraInfoTopicName>
-        <frameName>realsense_color_optical_frame</frameName>
-        <hackBaseline>0.07</hackBaseline>
-      </plugin>
-    </sensor>
+  <!-- Grasp-fix plugin. Robotiq parallel grasps are unreliable in Gazebo classic
+       (the cube slips out from between the finger pads). This plugin detects a
+       stable grip between the gripper links and an object, attaches it to the
+       palm with a temporary fixed joint, and releases when the gripper opens.
+       Provided by ros-noetic-roboticsgroup-upatras-gazebo-plugins. -->
+  <gazebo>
+    <plugin name="gazebo_grasp_fix" filename="libgazebo_grasp_fix.so">
+      <arm>
+        <arm_name>ur5_gripper</arm_name>
+        <!-- Gazebo lumps fixed-jointed links into their parent: the gripper base
+             (robotiq_arg2f_base_link) merges into wrist_3_link, and the
+             *_finger_tip links merge into the *_inner_finger links. So use the
+             real Gazebo link names here, not the URDF ones. -->
+        <palm_link>wrist_3_link</palm_link>
+        <gripper_link>left_inner_finger</gripper_link>
+        <gripper_link>right_inner_finger</gripper_link>
+      </arm>
+      <forces_angle_tolerance>120</forces_angle_tolerance>
+      <update_rate>15</update_rate>
+      <grip_count_threshold>1</grip_count_threshold>
+      <max_grip_count>3</max_grip_count>
+      <release_tolerance>0.008</release_tolerance>
+      <!-- Once a grip is detected, stop the fingers colliding with the object so
+           the position-controlled gripper can't crush/launch the light cube. -->
+      <disable_collisions_on_attach>true</disable_collisions_on_attach>
+      <contact_topic>__default_topic__</contact_topic>
+    </plugin>
   </gazebo>
 </robot>

File: ur5_with_robotiq_gripper/icl_ur5_setup_description/urdf/realsense.xacro (robot description, xacro)
@@ -1,59 +1,114 @@
 <?xml version="1.0"?>
 <robot xmlns:xacro="http://ros.org/wiki/xacro">
-  <!-- Physical link representing the camera body -->
-  <link name="realsense_link">
-    <visual>
-      <geometry>
-        <box size="0.025 0.09 0.025"/>
-      </geometry>
-      <material name="camera_grey">
-        <color rgba="0.5 0.5 0.5 1.0"/>
-      </material>
-    </visual>
-    <collision>
-      <geometry>
-        <box size="0.025 0.09 0.025"/>
-      </geometry>
-    </collision>
-    <inertial>
-      <mass value="0.072"/>
-      <inertia ixx="0.000001" ixy="0.0" ixz="0.0" iyy="0.000001" iyz="0.0" izz="0.000001"/>
-    </inertial>
-  </link>
-  <!-- Optical frame (standard ROS camera convention: x-right, y-down, z-forward) -->
-  <link name="realsense_color_optical_frame"/>
-  <joint name="realsense_optical_joint" type="fixed">
-    <parent link="realsense_link"/>
-    <child link="realsense_color_optical_frame"/>
-    <!-- Rotate from camera body frame to optical frame: x forward -> z forward, y left -> x right -->
-    <origin xyz="0 0 0" rpy="${-pi/2} 0 ${-pi/2}"/>
-  </joint>
-  <gazebo reference="realsense_link">
-    <sensor type="depth" name="realsense_camera">
-      <always_on>true</always_on>
-      <update_rate>30</update_rate>
-      <visualize>true</visualize>
-      <pose>0 0 0 0 0 0</pose>
-      <camera>
-        <horizontal_fov>1.3962634</horizontal_fov>
-        <image>
-          <width>640</width>
-          <height>480</height>
-          <format>R8G8B8</format>
-        </image>
-        <clip>
-          <near>0.1</near>
-          <far>5.0</far>
-        </clip>
-      </camera>
-      <plugin name="camera_controller" filename="libgazebo_ros_camera.so">
-        <robotNamespace>/ur5</robotNamespace>
-        <cameraName>realsense</cameraName>
-        <imageTopicName>camera/image_raw</imageTopicName>
-        <depthImageTopicName>camera/depth/image_raw</depthImageTopicName>
-        <cameraInfoTopicName>camera/camera_info</cameraInfoTopicName>
-        <frameName>realsense_color_optical_frame</frameName>
-      </plugin>
-    </sensor>
-  </gazebo>
+  <!-- Wrist-mounted depth (RGB-D) camera used for AprilTag detection.
+       Single source of truth for the camera link, mount joint, optical frame
+       and Gazebo sensor. Include this file and call the macro from the robot
+       xacro instead of duplicating the camera inline.
+       The Gazebo plugin publishes, in the ROS optical frame
+       'realsense_color_optical_frame':
+         /ur5/realsense/camera/image_raw         (sensor_msgs/Image, RGB)   <- AprilTag uses this
+         /ur5/realsense/camera/camera_info       (sensor_msgs/CameraInfo)   <- AprilTag uses this
+         /ur5/realsense/camera/depth/image_raw   (sensor_msgs/Image, depth) <- available for future use
+         /ur5/realsense/camera/depth/points      (sensor_msgs/PointCloud2)  <- available for future use -->
+  <xacro:macro name="realsense_camera" params="parent">
+    <!-- Physical camera body (dimensions unchanged) -->
+    <link name="realsense_link">
+      <visual>
+        <geometry>
+          <box size="0.025 0.09 0.025"/>
+        </geometry>
+        <material name="camera_grey">
+          <color rgba="0.5 0.5 0.5 1.0"/>
+        </material>
+      </visual>
+      <collision>
+        <geometry>
+          <box size="0.025 0.09 0.025"/>
+        </geometry>
+      </collision>
+      <inertial>
+        <mass value="0.072"/>
+        <inertia ixx="0.000001" ixy="0.0" ixz="0.0" iyy="0.000001" iyz="0.0" izz="0.000001"/>
+      </inertial>
+    </link>
+    <!-- Mount the camera on the wrist, offset up and forward -->
+    <joint name="realsense_joint" type="fixed">
+      <parent link="${parent}"/>
+      <child link="realsense_link"/>
+      <origin xyz="0 0.06 0.01" rpy="0 -1.5708 1.5708"/>
+    </joint>
+    <!-- Optical frame (ROS optical convention: X=right, Y=down, Z=forward) -->
+    <link name="realsense_color_optical_frame"/>
+    <joint name="realsense_optical_joint" type="fixed">
+      <parent link="realsense_link"/>
+      <child link="realsense_color_optical_frame"/>
+      <origin xyz="0 0 0" rpy="-1.5708 0 -1.5708"/>
+    </joint>
+    <!-- Two co-located Gazebo sensors on the same link/optical frame:
+         1) RGB camera (libgazebo_ros_camera.so) -> camera/image_raw +
+            camera/camera_info. The plain camera plugin publishes camera_info in
+            the RGB image callback, which is what AprilTag subscribes to.
+         2) Depth camera (libgazebo_ros_depth_camera.so) -> camera/depth/image_raw
+            + camera/depth/points, for future depth-based work.
+         A single depth plugin is intentionally NOT used for both: it only emits
+         camera_info when the depth stream is consumed, so AprilTag (RGB-only)
+         would receive 0 camera_info messages and never detect a tag. The depth
+         sensor's RGB-side outputs are renamed so they don't collide with (1). -->
+    <gazebo reference="realsense_link">
+      <sensor type="camera" name="realsense_color">
+        <always_on>true</always_on>
+        <update_rate>30</update_rate>
+        <visualize>true</visualize>
+        <camera>
+          <horizontal_fov>1.3962634</horizontal_fov>
+          <image>
+            <width>640</width>
+            <height>480</height>
+            <format>R8G8B8</format>
+          </image>
+          <clip>
+            <near>0.1</near>
+            <far>5.0</far>
+          </clip>
+        </camera>
+        <plugin name="realsense_color_controller" filename="libgazebo_ros_camera.so">
+          <robotNamespace>/ur5</robotNamespace>
+          <cameraName>realsense</cameraName>
+          <frameName>realsense_color_optical_frame</frameName>
+          <imageTopicName>camera/image_raw</imageTopicName>
+          <cameraInfoTopicName>camera/camera_info</cameraInfoTopicName>
+          <hackBaseline>0.07</hackBaseline>
+        </plugin>
+      </sensor>
+      <sensor type="depth" name="realsense_depth">
+        <always_on>true</always_on>
+        <update_rate>15</update_rate>
+        <camera>
+          <horizontal_fov>1.3962634</horizontal_fov>
+          <image>
+            <width>640</width>
+            <height>480</height>
+            <format>R8G8B8</format>
+          </image>
+          <clip>
+            <near>0.1</near>
+            <far>5.0</far>
+          </clip>
+        </camera>
+        <plugin name="realsense_depth_controller" filename="libgazebo_ros_depth_camera.so">
+          <robotNamespace>/ur5</robotNamespace>
+          <cameraName>realsense</cameraName>
+          <frameName>realsense_color_optical_frame</frameName>
+          <imageTopicName>camera/depth/color_image_raw</imageTopicName>
+          <cameraInfoTopicName>camera/depth/color_camera_info</cameraInfoTopicName>
+          <depthImageTopicName>camera/depth/image_raw</depthImageTopicName>
+          <depthImageCameraInfoTopicName>camera/depth/camera_info</depthImageCameraInfoTopicName>
+          <pointCloudTopicName>camera/depth/points</pointCloudTopicName>
+          <pointCloudCutoff>0.1</pointCloudCutoff>
+          <pointCloudCutoffMax>5.0</pointCloudCutoffMax>
+          <hackBaseline>0.07</hackBaseline>
+        </plugin>
+      </sensor>
+    </gazebo>
+  </xacro:macro>
 </robot>

File: ur5_with_robotiq_gripper/icl_ur5_setup_description/urdf/robotiq_arg2f_85_transmission.xacro (robot description, xacro)
@@ -5,4 +5,10 @@
       <type>transmission_interface/SimpleTransmission</type>
       <joint name="${prefix}finger_joint">
+        <!-- Position interface. NOTE: effort/force control was tried here to get
+             a gentle squeeze, but the Robotiq's underactuated closed-loop linkage
+             driven by the kinematic mimic-joint plugin does not track under
+             single-joint effort control (the gripper won't close). Position
+             control drives finger_joint to a setpoint and the mimic joints follow
+             consistently, so it is the reliable choice for this model. -->
         <hardwareInterface>hardware_interface/PositionJointInterface</hardwareInterface>
       </joint>
